Commit message: 添加日志 已经确认是plannerCloudCrop坐标系的问题

File: rm_simulation/pb_rm_simulation/urdf/simulation_waking_robot.xacro (robot description, xacro)
@@ -14,5 +14,5 @@
   <xacro:arg name="xyz" default="0.12 0.0 0.175" />
   <xacro:arg name="rpy" default="0 0 0" />
-  <link name="dummy"/>
+  <!-- <link name="dummy"/> -->
   <link name="base_link">
     <visual>
@@ -33,8 +33,8 @@
     <xacro:default_inertial mass="8.2"/>
   </link>
-  <joint name="dummy_joint" type="fixed">
+  <!-- <joint name="dummy_joint" type="fixed">
      <parent link="dummy"/>
      <child link="base_link"/>
-  </joint>
+  </joint> -->
   <link name="wheel_1">
     <visual>

Commit message: 将控制器输出的速度限制为两位小数

File: rm_simulation/pb_rm_simulation/urdf/simulation_waking_robot.xacro (robot description, xacro)
@@ -12,5 +12,5 @@
   </xacro:macro>
   <!-- base_link to livox_frame -->
-  <xacro:arg name="xyz" default="0.12 0.0 0.175" />
+  <xacro:arg name="xyz" default="0.5 0.0 0.35" />
   <xacro:arg name="rpy" default="0 0 0" />
   <!-- <link name="dummy"/> -->
@@ -18,5 +18,5 @@
     <visual>
       <geometry>
-        <box size="0.2 .3 .1"/>
+        <box size="0.5 0.3 0.2"/>
       </geometry>
       <origin rpy="0 0 ${PI/2}" xyz="0 0 0.05"/>
@@ -27,5 +27,5 @@
     <collision>
       <geometry>
-        <box size="0.2 .3 0.1"/>
+        <box size="0.5 .3 0.2"/>
       </geometry>
       <origin rpy="0 0 ${PI/2}" xyz="0 0 0.05"/>

Commit message: 可以使用,就是没有那么丝滑

File: rm_simulation/pb_rm_simulation/urdf/simulation_waking_robot.xacro (robot description, xacro)
@@ -12,5 +12,5 @@
   </xacro:macro>
   <!-- base_link to livox_frame -->
-  <xacro:arg name="xyz" default="0.5 0.0 0.35" />
+  <xacro:arg name="xyz" default="0.12 0.0 0.2" />
   <xacro:arg name="rpy" default="0 0 0" />
   <!-- <link name="dummy"/> -->
@@ -18,5 +18,5 @@
     <visual>
       <geometry>
-        <box size="0.5 0.3 0.2"/>
+        <box size="0.2 0.3 0.1"/>
       </geometry>
       <origin rpy="0 0 ${PI/2}" xyz="0 0 0.05"/>

Commit message: 解决仿真环境时间戳的问题

File: rm_simulation/pb_rm_simulation/urdf/simulation_waking_robot.xacro (robot description, xacro)
@@ -139,4 +139,32 @@
     <parent link="base_link"/>
     <child link="imu_link"/>
+  </joint>
+  <!-- Depth Camera Link -->
+  <link name="camera_link">
+    <visual>
+      <geometry>
+        <box size="0.05 0.05 0.05"/>
+      </geometry>
+      <material name="blue">
+        <color rgba="0 0 1 1"/>
+      </material>
+    </visual>
+    <collision>
+      <geometry>
+        <box size="0.05 0.05 0.05"/>
+      </geometry>
+    </collision>
+    <inertial>
+      <mass value="0.1"/>
+      <inertia ixx="1e-4" ixy="0" ixz="0"
+              iyy="1e-4" iyz="0" izz="1e-4"/>
+    </inertial>
+  </link>
+  <!-- Mount camera to base_link -->
+  <joint name="camera_joint" type="fixed">
+    <parent link="base_link"/>
+    <child link="camera_link"/>
+    <!-- camera 放在机器人前面 0.15m，稍微抬起 0.15m -->
+    <origin xyz="0.15 0 0.15" rpy="0 0 0"/>
   </joint>
   <!-- IMU -->
@@ -212,4 +240,39 @@
     </plugin>
   </gazebo>
+  <gazebo reference="camera_link">
+  <sensor name="depth_camera" type="depth">
+    <update_rate>30</update_rate>
+    <always_on>true</always_on>
+    <visualize>true</visualize>
+    <!-- 深度相机参数 -->
+    <camera>
+      <horizontal_fov>1.047</horizontal_fov> <!-- 60° -->
+      <image>
+        <width>640</width>
+        <height>480</height>
+        <format>R8G8B8</format>
+      </image>
+      <clip>
+        <near>0.1</near>
+        <far>10.0</far>
+      </clip>
+    </camera>
+    <!-- ROS 插件输出 Depth + RGB -->
+    <plugin name="camera_plugin" filename="libgazebo_ros_camera.so">
+      <ros>
+        <namespace>/</namespace>
+        <remapping>camera:=camera/color</remapping>
+      </ros>
+      <frame_name>camera_link</frame_name>
+    </plugin>
+    <plugin name="depth_camera_plugin" filename="libgazebo_ros_depth_camera.so">
+      <ros>
+        <namespace>/</namespace>
+        <remapping>camera/depth/image_raw:=camera/depth/image_raw</remapping>
+      </ros>
+      <frame_name>camera_link</frame_name>
+    </plugin>
+    </sensor>
+  </gazebo>
   <!-- mid360_imu plugin -->
   <!-- https://github.com/ros-simulation/gazebo_ros_pkgs/wiki/ROS-2-Migration:-IMU-Sensors -->
